File: DRV8711.sch (KiCad schematic (older format))
At the start: 7 parts, among them P1 CONN_01X04, U1 DRV8711

Commit message: KiCAD version updated
Parts:
- C1, C2, C3, C4, C5: symbol C_Small -> oh_stepper_driver-rescue:C_Small
- P1: symbol CONN_01X04 -> oh_stepper_driver-rescue:CONN_01X04
- U1: symbol DRV8711 -> drv8711:DRV8711
Changed lines of the file:
@@
-EESchema Schematic File Version 2
-LIBS:csd18531q5a
-LIBS:drv8711
-LIBS:stm32f446_lqfp64
-LIBS:abm8g
-LIBS:oh_stepper_driver-rescue
-LIBS:power
-LIBS:device
-LIBS:transistors
-LIBS:conn
-LIBS:linear
-LIBS:regul
-LIBS:74xx
-LIBS:cmos4000
-LIBS:adc-dac
-LIBS:memory
-LIBS:xilinx
-LIBS:microcontrollers
-LIBS:dsp
-LIBS:microchip
-LIBS:analog_switches
-LIBS:motorola
-LIBS:texas
-LIBS:intel
-LIBS:audio
-LIBS:interface
-LIBS:digital-audio
-LIBS:philips
-LIBS:display
-LIBS:cypress
-LIBS:siliconi
-LIBS:opto
-LIBS:atmel
-LIBS:contrib
-LIBS:valves
-LIBS:tja1050
-LIBS:as5047d
+EESchema Schematic File Version 4
 LIBS:oh_stepper_driver-cache
 EELAYER 26 0
@@
 $EndDescr
 $Comp
-L GND #PWR26
+L power:GND #PWR26
 U 1 1 587A445C
 P 3950 5000
@@
 BOUT2
 $Comp
-L C_Small C5
+L oh_stepper_driver-rescue:C_Small C5
 U 1 1 587A4D91
 P 5050 4600
@@
 $EndComp
 $Comp
-L GND #PWR27
+L power:GND #PWR27
 U 1 1 587A506C
 P 5050 4800
@@
 $EndComp
 $Comp
-L C_Small C1
+L oh_stepper_driver-rescue:C_Small C1
 U 1 1 587A2B22
 P 2150 3050
@@
 $EndComp
 $Comp
-L C_Small C3
+L oh_stepper_driver-rescue:C_Small C3
 U 1 1 587A2EDF
 P 2500 2500
@@
 $EndComp
 $Comp
-L C_Small C2
+L oh_stepper_driver-rescue:C_Small C2
 U 1 1 587A2F5D
 P 2300 2300
@@
 $EndComp
 $Comp
-L C_Small C4
+L oh_stepper_driver-rescue:C_Small C4
 U 1 1 587A2F63
 P 2600 3050
@@
 	3800 4900 3800 4950
 Wire Wire Line
-	3800 4950 4100 4950
+	3800 4950 3900 4950
 Wire Wire Line
 	4100 4950 4100 4900
@@
 	2900 4600 2525 4600
 $Comp
-L GND #PWR25
+L power:GND #PWR25
 U 1 1 587A44CC
 P 2150 3225
@@
 	2600 3175 2150 3175
 Wire Wire Line
-	2150 3150 2150 3225
+	2150 3150 2150 3175
 Connection ~ 2150 3175
 $Comp
-L VM #PWR24
+L oh_stepper_driver-rescue:VM #PWR24
 U 1 1 587A4A3A
 P 2150 2100
@@
 	2300 2650 2300 2400
 Wire Wire Line
-	2150 2100 2150 2750
+	2150 2100 2150 2150
 Wire Wire Line
 	2150 2150 2300 2150
@@
 Connection ~ 2150 2150
 $Comp
-L DRV8711 U1
+L drv8711:DRV8711 U1
 U 1 1 587A59C2
 P 3800 3450
@@
 	8750 3100 9300 3100
 $Comp
-L CONN_01X04 P1
+L oh_stepper_driver-rescue:CONN_01X04 P1
 U 1 1 587B6637
 P 9650 2800
@@
 Text HLabel 2525 4600 0    60   Output ~ 0
 STALLn
+Wire Wire Line
+	4000 4950 4100 4950
+Wire Wire Line
+	3900 4950 3950 4950
+Wire Wire Line
+	3950 4950 4000 4950
+Wire Wire Line
+	2150 3175 2150 3225
+Wire Wire Line
+	2150 2150 2150 2750
 $EndSCHEMATC
