File: FETs.sch (KiCad schematic (older format))
At the start: 20 parts, among them Q1 CSD18531Q5A, Q2 CSD18531Q5A, Q3 CSD18531Q5A, Q4 CSD18531Q5A, Q5 CSD18531Q5A, Q6 CSD18531Q5A, Q7 CSD18531Q5A, Q8 CSD18531Q5A

Commit message: KiCAD version updated
Parts:
- Q1, Q2, Q3, Q4, Q5, Q6, Q7, Q8: symbol CSD18531Q5A -> csd18531q5a:CSD18531Q5A
- R1, R10, R11, R12, R2, R3, R4, R5, R6, R7, R8, R9: symbol R_Small -> oh_stepper_driver-rescue:R_Small
